Commit message: Created preliminary launch file for teleop

File: ROSMaster/worlds/models/robot/urdf/rover.urdf (robot description, URDF)
Before this commit: robot rover, 9 links, 7 joints
Links:
- removed link us1_link
- removed link us2_link
- removed link us3_link
- removed link us4_link
- added link US1_link, mass 0.0451494993409843; collision mesh filename=package://worlds/models/robot/meshes/US1_link.STL; visual mesh filename=package://worlds/models/robot/meshes/US1_link.STL
- added link US2_link, mass 0.0451494993409843; collision mesh filename=package://worlds/models/robot/meshes/US2_link.STL; visual mesh filename=package://worlds/models/robot/meshes/US2_link.STL
- added link US3_link, mass 0.0451494993409843; collision mesh filename=package://worlds/models/robot/meshes/US3_link.STL; visual mesh filename=package://worlds/models/robot/meshes/US3_link.STL
- added link US4_link, mass 0.0451494993409843; collision mesh filename=package://worlds/models/robot/meshes/US4_link.STL; visual mesh filename=package://worlds/models/robot/meshes/US4_link.STL
- link base_link: mass 0.229882969798051 -> 1.6; geometry collision mesh filename=package://worlds/models/robot/meshes/base_link.STL; visual mesh filename=package://worlds/models/robot/meshes/base_link.STL
- link lidar_link: mass 0.21166 -> 0.2; geometry collision mesh filename=package://worlds/models/robot/meshes/lidar_link.STL; visual mesh filename=package://worlds/models/robot/meshes/lidar_link.STL
- link wheel1_link: mass 0.060901 -> 0.0609005806210085; geometry collision mesh filename=package://worlds/models/robot/meshes/wheel1_link.STL; visual mesh filename=package://worlds/models/robot/meshes/wheel1_link.STL
- link wheel2_link: mass 0.060901 -> 0.0609005806210085; geometry collision mesh filename=package://worlds/models/robot/meshes/wheel2_link.STL; visual mesh filename=package://worlds/models/robot/meshes/wheel2_link.STL
- link wheel3_link: mass 0.060901 -> 0.0609005806210086; geometry collision mesh filename=package://worlds/models/robot/meshes/wheel3_link.STL; visual mesh filename=package://worlds/models/robot/meshes/wheel3_link.STL
Joints:
- removed joint us1_joint
- removed joint us2_joint
- removed joint us3_joint
- removed joint us4_joint
- added joint US1_joint: type fixed, parent base_link, child US1_link, origin xyz=0.087637 -6.35E-05 0.14173 rpy=0 0 0, axis 0 0 0
- added joint US2_joint: type fixed, parent base_link, child US2_link, origin xyz=0 -0.087637 0.14173 rpy=0 0 -1.5708, axis 0 0 0
- added joint US3_joint: type fixed, parent base_link, child US3_link, origin xyz=-0.087637 -6.35E-05 0.14173 rpy=0 0 -3.1416, axis 0 0 0
- added joint US4_joint: type fixed, parent base_link, child US4_link, origin xyz=0 0.087637 0.14173 rpy=0 0 1.5708, axis 0 0 0
- added joint wheel3_joint: type continuous, parent base_link, child wheel3_link, origin xyz=-0.091567 0 0 rpy=0 0 -1.5708, axis 0 1 0, limit effort=1000 velocity=8.59
- joint lidar_joint: axis 0 1 0 -> 0 0 1; limit (none) -> effort=1000 velocity=42; origin xyz=0.0067498 -0.036576 0.18339 rpy=1.5708 0 -1.1777 -> xyz=0.00674979600000013 -0.036576 0.238388 rpy=0 0 0
- joint wheel1_joint: axis 0 0 1 -> 0 1 0; limit (none) -> effort=1000 velocity=8.59; origin xyz=0.048665 0.08429 0 rpy=-1.5708 -0.38253 -0.5236 -> xyz=0.045784 0.079299 0 rpy=0 0 2.618
- joint wheel2_joint: axis 0 0 1 -> 0 1 0; child wheel3_link -> wheel2_link; limit (none) -> effort=1000 velocity=8.59; origin xyz=-0.091567 0 0 rpy=-1.5708 -0.39309 1.5708 -> xyz=0.0457835000000003 -0.0792993481483295 0 rpy=0 0 0.523598775598303

Commit message: Fix Rviz configs

File: ROSMaster/worlds/models/robot/urdf/rover.urdf (robot description, URDF)
Before this commit: robot rover, 9 links, 8 joints
Links:
- removed link US1_link
- removed link US2_link
- removed link US3_link
- removed link US4_link
Joints:
- removed joint US1_joint
- removed joint US2_joint
- removed joint US3_joint
- removed joint US4_joint

Commit message: Just got to MC on Sunday

File: ROSMaster/worlds/models/robot/urdf/rover.urdf (robot description, URDF)
Before this commit: robot rover, 5 links, 4 joints
Joints:
- joint lidar_joint: origin xyz=0.00674979600000013 -0.036576 0.238388 rpy=0 0 0 -> xyz=0.0 0.0 0.238388 rpy=0 0 0
